Commit message: add imu_link

File: src/velodyne_wt61c/urdf/sensor_suite.urdf (robot description, URDF)
Before this commit: robot sensor_suite, 3 links, 2 joints
Links:
- added link imu_link
Joints:
- added joint imu_link_joint: type fixed, parent base_link, child imu_link, origin xyz=0 0 0 rpy=0 0 0
- joint wt61c_uart_joint: parent base_link -> imu_link

Commit message: modify frame

File: src/velodyne_wt61c/urdf/sensor_suite.urdf (robot description, URDF)
Before this commit: robot sensor_suite, 4 links, 3 joints
Links:
- added link lidar_link
Joints:
- added joint lidar_joint: type fixed, parent base_link, child lidar_link, origin xyz=0 0 0 rpy=0 0 0
- joint imu_link_joint: parent base_link -> lidar_link
- joint velodyne_joint: parent base_link -> lidar_link
